File: design/source/kicad/cicada-2g/cicada-2g.sch (KiCad schematic (older format))
At the start: 60 parts, among them J2 Host, J3 USB_OTG, J4 IPX, J5 DNP IPX, P1 SK-C793, Q1 2N7002, U1 74LVC1G17, U2 USBLC6-2SC6, U3 M3406-ADJ, U4 SIM800C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

Commit message: Clean up the component libraries
Parts:
- L4: footprint Inductor_SMD:L_Taiyo-Yuden_NR-40xx_HandSoldering -> cicada-footprints:L_4030_Handsoldering
- P1: footprint sk-c793:SK-C793 -> cicada-footprints:SK-C793
Changed lines of the file:
@@
 F 0 "L4" V 3950 9300 50  0000 C CNN
 F 1 "3.3uH 1A" V 3850 9200 50  0000 C CNN
-F 2 "Inductor_SMD:L_Taiyo-Yuden_NR-40xx_HandSoldering" H 3750 9350 50  0001 C CNN
+F 2 "cicada-footprints:L_4030_Handsoldering" H 3750 9350 50  0001 C CNN
 F 3 "~" H 3750 9350 50  0001 C CNN
 F 4 "FPI0403F-3R3M" H -2750 5600 50  0001 C CNN "MPN"
@@
 F 0 "P1" H 11500 8400 50  0000 C CNN
 F 1 "SK-C793" H 11600 8300 50  0000 C CNN
-F 2 "sk-c793:SK-C793" H 11600 8650 50  0001 C CNN
+F 2 "cicada-footprints:SK-C793" H 11600 8650 50  0001 C CNN
 F 3 "" H 11600 8650 50  0001 C CNN
 F 4 "SK-C793" H 7000 -750 50  0001 C CNN "MPN"

Commit message: Update the library directory structure to match other Okra projects
Parts:
- J4, J5: footprint Connector_Coaxial:U.FL_Molex_MCRF_73412-0110_Vertical -> cicada-footprints:U.FL_Molex_MCRF_73412-0110_Vertical
Connections:
- wire segments 224 -> 229
- no-connect marks 21 -> 29
Other:
- moved on the sheet: D10, D5, J3, R14
