File: design/source/kicad/cicada-2g/P-1000010_Okra Cicada 2G PCBA.kicad_sch (KiCad schematic)
At the start: 67 parts

Commit message: Make PCB revisions dynamic
Other:
- title: Ciacada 2G -> Cicada 2G
Changed lines of the file:
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@@
   (paper "A3")
   (title_block
-    (title "Ciacada 2G")
+    (title "Cicada 2G")
     (date "2020-05-15")
-    (rev "2.0")
+    (rev "${PROJECT_REVISION}")
     (company "Alexey Zaytsev / Okra Solar")
   )
