File: design/source/kicad/cicada-4g/P-1000011_Okra Cicada 4G PCBA.kicad_sch (KiCad schematic)
At the start: 96 parts

Commit message: Make PCB revisions dynamic
Other:
- title: Ciacada 4G -> Cicada 4G
Changed lines of the file:
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@@
   (paper "A3")
   (title_block
-    (title "Ciacada 4G")
+    (title "Cicada 4G")
     (date "2020-05-15")
-    (rev "2.0")
+    (rev "${PROJECT_REVISION}")
     (company "Alexey Zaytsev / Okra Solar")
   )
