File: design/source/kicad/cicada-4g/P-1000011_Okra Cicada 4G PCBA.kicad_pcb (KiCad board)
At the start: 4 copper layers, 40 x 65 mm, 95 parts, among them J2 Host, J3 USB_OTG, J4 IPX, J5 IPX, J6 IPX, J7 Conn_01x04, J8 IPX, P1 SK-C793, Q1 NMOS, Q2 NMOS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

Commit message: Use dynamic revisions in PCBs
Other:
- board text added: "Cicada 4G v${PROJECT_REVISION}"
- board text removed: "Cicada 4G v2.0"
Changed lines of the file:
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@@
     (effects (font (size 1.2 1.2) (thickness 0.17)) (justify right))
   )
-  (gr_text "Cicada 4G v2.0" (at 133 84.15 90) (layer "F.SilkS")
+  (gr_text "Cicada 4G v${PROJECT_REVISION}" (at 133 84.15 90) (layer "F.SilkS")
     (effects (font (size 1.8 1.8) (thickness 0.35) italic))
   )
